File: blizzard_projects/Blizzard_Board/main.sch (EAGLE design)
At the start: 81 parts, among them J1 XH_4POS_DEV, J2 XH_5POS_DEV, J3 XH_4POS_DEV, J4 XH_8POS_DEV, J5 XH_5POS_DEV, Q1 s8050(NPN), Q2 S8050(NPN), Q3 N2222, Q4 N2222, U1 USB_TO_UART_DEV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

Commit message: started tracing
Parts:
- removed R34, R38: 0, blizzard_common_1:0805_RES_DEV
- added J6, J7: XH_2POS_DEV, blizzard_common_1:XH_2POS_DEV
- J4: value XH_8POS_DEV -> XH_6POS_DEV; device blizzard_common_1:XH_8POS_DEV -> blizzard_common_1:XH_6POS_DEV
Connections:
- removed net N$1 (its old number): U1.DCD
- removed net N$11 (its old number): U1.!SUSPEND
- removed net N$13: U1.NC1
- removed net N$14: U1.NC2
- removed net N$15: U1.NC3
- removed net N$16: U1.NC4
- removed net N$17: U1.NC5
- removed net N$18: U1.NC6
- removed net N$19: U1.NC7
- removed net N$2 (its old number): U1.RI
- removed net N$20: U1.NC8
- removed net N$21: U1.NC9
- removed net N$22: U1.NC10
- removed net N$23: U1.CTS
- removed net N$27: U1.DSR
- removed net N$45: J4.P$3, R34.P$2
- removed net N$46: J4.P$4, R35.P$2
- removed net N$48: J4.P$6, R37.P$2
- removed net N$49: J4.P$7, R38.P$2
- removed net N$50: J4.P$8, R39.P$2
- net 3.3V: now also J7.P$1
- net 5V: now also J6.P$1
- net GND: now also J6.P$2, J7.P$2, S1.3, S1.4, S2.3, S2.4; no longer S1.P$2, S2.P$2
- net IO17: no longer R38.P$1
- net IO27: no longer R34.P$1
- net N$10: now also J4.P$4, R37.P$2; no longer U1.NC0
- net N$12: now also J4.P$6, R35.P$2; no longer U1.SUSPEND
- net N$25: now also S1.1, S1.2; no longer S1.P$1
- net N$29: now also S2.1, S2.2; no longer S2.P$1
- net N$9: now also J4.P$3, R39.P$2; no longer U1.!RST
Other:
- note added: "+"
- note added: "-"
- note added: "3.3V Out"
- note added: "5V In"
- note added: "Blizzard Lighting LLC"
- note added: "Date: 8.2.17"
- note added: "Designed By: Christian Krueger"
- note added: "Eth CRS"
- note added: "Eth Pow"
- note added: "REV: 0.1"
- note added: "Sheet: 1/1"
- note added: "Title: Blizzard Board"
- moved on the sheet: C5, C6, L1, R35, R37, R39, U2

Commit message: v1 out to order
Parts:
- added R34, R38, R40: 0, blizzard_common_1:0805_RES_DEV
- R4, R5: value 0805_RES_DEV -> 12K
Connections:
- removed net N$31: U4.XTAL2
- new net N$13: R38.P$2, U3.IO12
- new net N$14: R40.P$2, U3.IO15
- net 5V: now also J3.P$4
- net GND: now also R34.P$2
- net IO12: now also R38.P$1; no longer U3.IO12
- net IO15: now also R40.P$1; no longer U3.IO15
- net IO16: now also R39.P$1; no longer R37.P$1
- net IO4: now also R37.P$1; no longer R36.P$1
- net IO5: now also R36.P$1; no longer R39.P$1
- net N$8: now also R34.P$1
Other:
- moved on the sheet: J2, J5

Commit message: waiting on first order
Parts:
- C12, C13, C14, C17: value 104 -> 0.1uF
- C15: value 0805_CAP_DEV -> 470pF
- C16: value 0805_CAP_DEV -> 1uF
- C18: value 0805_CAP_DEV -> 0.022uF
Other:
- note added: "Do not populate"
Changed lines of the file:
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@@
 <setting verticaltext="up"/>
 </settings>
-<grid distance="0.1" unitdist="inch" unit="mm" style="lines" multiple="1" display="yes" altdistance="0.01" altunitdist="inch" altunit="mm"/>
+<grid distance="0.1" unitdist="inch" unit="inch" style="lines" multiple="1" display="no" altdistance="0.01" altunitdist="inch" altunit="inch"/>
 <layers>
 <layer number="1" name="Top" color="4" fill="1" visible="no" active="no"/>
@@
 <part name="R9" library="blizzard_common_1" deviceset="0805_RES_DEV" device="" value="33"/>
 <part name="R10" library="blizzard_common_1" deviceset="0805_RES_DEV" device="" value="33"/>
-<part name="C12" library="blizzard_common_1" deviceset="0805_CAP_DEV" device="" value="104"/>
-<part name="C13" library="blizzard_common_1" deviceset="0805_CAP_DEV" device="" value="104"/>
+<part name="C12" library="blizzard_common_1" deviceset="0805_CAP_DEV" device="" value="0.1uF"/>
+<part name="C13" library="blizzard_common_1" deviceset="0805_CAP_DEV" device="" value="0.1uF"/>
 <part name="L2" library="blizzard_common_1" deviceset="0805_IND_DEV" device="" value="FB"/>
 <part name="R11" library="blizzard_common_1" deviceset="0805_RES_DEV" device="" value="1.5K"/>
-<part name="C14" library="blizzard_common_1" deviceset="0805_CAP_DEV" device="" value="104"/>
-<part name="C15" library="blizzard_common_1" deviceset="0805_CAP_DEV" device=""/>
-<part name="C16" library="blizzard_common_1" deviceset="0805_CAP_DEV" device=""/>
+<part name="C14" library="blizzard_common_1" deviceset="0805_CAP_DEV" device="" value="0.1uF"/>
+<part name="C15" library="blizzard_common_1" deviceset="0805_CAP_DEV" device="" value="470pF"/>
+<part name="C16" library="blizzard_common_1" deviceset="0805_CAP_DEV" device="" value="1uF"/>
 <part name="R12" library="blizzard_common_1" deviceset="0805_RES_DEV" device="" value="12.1K"/>
 <part name="Y1" library="blizzard_board" deviceset="OSC_DEV" device="" value="50MHz"/>
@@
 <part name="R16" library="blizzard_common_1" deviceset="0805_RES_DEV" device="" value="33"/>
 <part name="R17" library="blizzard_common_1" deviceset="0805_RES_DEV" device="" value="4.7K"/>
-<part name="C17" library="blizzard_common_1" deviceset="0805_CAP_DEV" device="" value="104"/>
+<part name="C17" library="blizzard_common_1" deviceset="0805_CAP_DEV" device="" value="0.1uF"/>
 <part name="R18" library="blizzard_common_1" deviceset="0805_RES_DEV" device="" value="4.7K"/>
 <part name="R19" library="blizzard_common_1" deviceset="0805_RES_DEV" device="" value="10"/>
@@
 <part name="R22" library="blizzard_common_1" deviceset="0805_RES_DEV" device="" value="10"/>
 <part name="R23" library="blizzard_common_1" deviceset="0805_RES_DEV" device="" value="0"/>
-<part name="C18" library="blizzard_common_1" deviceset="0805_CAP_DEV" device=""/>
+<part name="C18" library="blizzard_common_1" deviceset="0805_CAP_DEV" device="" value="0.022uF"/>
 <part name="R24" library="blizzard_common_1" deviceset="0805_RES_DEV" device="" value="49.9"/>
 <part name="R25" library="blizzard_common_1" deviceset="0805_RES_DEV" device="" value="49.9"/>
@@
 <wire x1="231.14" y1="-93.98" x2="231.14" y2="-81.28" width="0.1524" layer="97"/>
 <text x="-116.84" y="15.24" size="1.6764" layer="97">NC</text>
+<text x="-96.52" y="2.54" size="1.778" layer="97" rot="R180">Do not populate</text>
+<wire x1="-111.76" y1="2.54" x2="-116.84" y2="10.16" width="0.1524" layer="97"/>
+<wire x1="-116.84" y1="10.16" x2="-116.84" y2="8.128" width="0.1524" layer="97"/>
+<wire x1="-116.84" y1="8.128" x2="-114.808" y2="9.398" width="0.1524" layer="97"/>
+<wire x1="-114.808" y1="9.398" x2="-116.84" y2="10.16" width="0.1524" layer="97"/>
 </plain>
 <instances>

Commit message: REV 1.2
Connections:
- new net NC: J2.P$2, J5.P$2
- net 3.3V: no longer J2.P$2, J5.P$2
- net IO32: now also R33.P$1; no longer J2.P$3, J5.P$3
- net IO34: now also J2.P$3, J5.P$3; no longer R33.P$1
Other:
- note removed: "Do not populate"
- note removed: "NC"
Changed lines of the file:
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@@
 <text x="40.64" y="172.72" size="1.6764" layer="97">AnyFi B</text>
 <text x="40.64" y="170.18" size="1.6764" layer="97">Extra</text>
-<text x="40.64" y="167.64" size="1.6764" layer="97">Extra</text>
+<text x="40.64" y="162.56" size="1.6764" layer="97">Extra</text>
 <text x="40.64" y="152.4" size="1.6764" layer="97">Eth CRS</text>
 <text x="109.22" y="101.6" size="1.6764" layer="97" rot="R90">Extra</text>
@@
 <text x="139.7" y="157.48" size="1.6764" layer="97">Extra</text>
 <text x="40.64" y="165.1" size="1.6764" layer="97">AnyFi R</text>
-<text x="40.64" y="162.56" size="1.6764" layer="97">AnyFi G</text>
+<text x="40.64" y="167.64" size="1.6764" layer="97">AnyFi G</text>
 <text x="40.64" y="160.02" size="1.6764" layer="97">AnyFi K</text>
 <text x="40.64" y="157.48" size="1.6764" layer="97">Eth RXD0</text>
@@
 <wire x1="228.6" y1="-104.14" x2="228.6" y2="-93.98" width="0.1524" layer="97"/>
 <wire x1="231.14" y1="-93.98" x2="231.14" y2="-81.28" width="0.1524" layer="97"/>
-<text x="-116.84" y="15.24" size="1.6764" layer="97">NC</text>
-<text x="-96.52" y="2.54" size="1.778" layer="97" rot="R180">Do not populate</text>
-<wire x1="-111.76" y1="2.54" x2="-116.84" y2="10.16" width="0.1524" layer="97"/>
-<wire x1="-116.84" y1="10.16" x2="-116.84" y2="8.128" width="0.1524" layer="97"/>
-<wire x1="-116.84" y1="8.128" x2="-114.808" y2="9.398" width="0.1524" layer="97"/>
-<wire x1="-114.808" y1="9.398" x2="-116.84" y2="10.16" width="0.1524" layer="97"/>
 </plain>
 <instances>
@@
 <label x="187.96" y="-15.24" size="1.6764" layer="95" rot="R270" xref="yes"/>
 </segment>
-<segment>
-<wire x1="215.9" y1="127" x2="246.38" y2="127" width="0.1524" layer="91"/>
-<wire x1="246.38" y1="127" x2="246.38" y2="116.84" width="0.1524" layer="91"/>
-<pinref part="J5" gate="G$1" pin="P$2"/>
-<wire x1="246.38" y1="116.84" x2="248.92" y2="116.84" width="0.1524" layer="91"/>
-<pinref part="J2" gate="G$1" pin="P$2"/>
-<wire x1="220.98" y1="116.84" x2="215.9" y2="116.84" width="0.1524" layer="91"/>
-<label x="210.82" y="116.84" size="1.6764" layer="95" rot="R180" xref="yes"/>
-<wire x1="215.9" y1="116.84" x2="210.82" y2="116.84" width="0.1524" layer="91"/>
-<wire x1="215.9" y1="127" x2="215.9" y2="116.84" width="0.1524" layer="91"/>
-<junction x="215.9" y="116.84"/>
-</segment>
 </net>
 <net name="5V" class="0">
@@
 </segment>
 <segment>
-<pinref part="R33" gate="G$1" pin="P$1"/>
-<wire x1="238.76" y1="200.66" x2="233.68" y2="200.66" width="0.1524" layer="91"/>
-<label x="233.68" y="200.66" size="1.6764" layer="95" rot="R180" xref="yes"/>
+<pinref part="J2" gate="G$1" pin="P$3"/>
+<wire x1="220.98" y1="114.3" x2="213.36" y2="114.3" width="0.1524" layer="91"/>
+<label x="203.2" y="114.3" size="1.778" layer="95" rot="R180" xref="yes"/>
+<pinref part="J5" gate="G$1" pin="P$3"/>
+<wire x1="213.36" y1="114.3" x2="203.2" y2="114.3" width="0.1524" layer="91"/>
+<wire x1="248.92" y1="114.3" x2="243.84" y2="114.3" width="0.1524" layer="91"/>
+<wire x1="243.84" y1="114.3" x2="243.84" y2="129.54" width="0.1524" layer="91"/>
+<wire x1="243.84" y1="129.54" x2="213.36" y2="129.54" width="0.1524" layer="91"/>
+<wire x1="213.36" y1="129.54" x2="213.36" y2="114.3" width="0.1524" layer="91"/>
+<junction x="213.36" y="114.3"/>
 </segment>
 </net>
@@
 </segment>
 <segment>
-<pinref part="J2" gate="G$1" pin="P$3"/>
-<wire x1="220.98" y1="114.3" x2="213.36" y2="114.3" width="0.1524" layer="91"/>
-<label x="203.2" y="114.3" size="1.6764" layer="95" rot="R180" xref="yes"/>
-<wire x1="213.36" y1="114.3" x2="203.2" y2="114.3" width="0.1524" layer="91"/>
-<wire x1="213.36" y1="114.3" x2="213.36" y2="129.54" width="0.1524" layer="91"/>
-<junction x="213.36" y="114.3"/>
-<wire x1="213.36" y1="129.54" x2="243.84" y2="129.54" width="0.1524" layer="91"/>
-<wire x1="243.84" y1="129.54" x2="243.84" y2="114.3" width="0.1524" layer="91"/>
-<pinref part="J5" gate="G$1" pin="P$3"/>
-<wire x1="243.84" y1="114.3" x2="248.92" y2="114.3" width="0.1524" layer="91"/>
+<pinref part="R33" gate="G$1" pin="P$1"/>
+<wire x1="238.76" y1="200.66" x2="233.68" y2="200.66" width="0.1524" layer="91"/>
+<label x="233.68" y="200.66" size="1.778" layer="95" rot="R180" xref="yes"/>
 </segment>
 </net>
@@
 </segment>
 </net>
+<net name="NC" class="0">
+<segment>
+<wire x1="215.9" y1="127" x2="246.38" y2="127" width="0.1524" layer="91"/>
+<wire x1="246.38" y1="127" x2="246.38" y2="116.84" width="0.1524" layer="91"/>
+<pinref part="J5" gate="G$1" pin="P$2"/>
+<wire x1="246.38" y1="116.84" x2="248.92" y2="116.84" width="0.1524" layer="91"/>
+<pinref part="J2" gate="G$1" pin="P$2"/>
+<wire x1="220.98" y1="116.84" x2="215.9" y2="116.84" width="0.1524" layer="91"/>
+<label x="210.82" y="116.84" size="1.6764" layer="95" rot="R180" xref="yes"/>
+<wire x1="215.9" y1="116.84" x2="210.82" y2="116.84" width="0.1524" layer="91"/>
+<wire x1="215.9" y1="127" x2="215.9" y2="116.84" width="0.1524" layer="91"/>
+<junction x="215.9" y="116.84"/>
+</segment>
+</net>

Commit message: version 1.2
Parts:
- removed R29, R30: 0, blizzard_common_1:0805_RES_DEV
Connections:
- removed net N$39: J1.P$3, R30.P$2
- removed net N$40: J1.P$2, R29.P$2
- net DMX+: now also J1.P$3; no longer R30.P$1
- net DMX-: now also J1.P$2; no longer R29.P$1
Changed lines of the file:
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@@
 <part name="Q3" library="blizzard_common_0" deviceset="NPN_N2222_DEV" device="" value="N2222"/>
 <part name="R27" library="blizzard_common_1" deviceset="0805_RES_DEV" device="" value="1K"/>
-<part name="R29" library="blizzard_common_1" deviceset="0805_RES_DEV" device="" value="0"/>
-<part name="R30" library="blizzard_common_1" deviceset="0805_RES_DEV" device="" value="0"/>
 <part name="Q4" library="blizzard_common_0" deviceset="NPN_N2222_DEV" device="" value="N2222"/>
 <part name="R31" library="blizzard_common_1" deviceset="0805_RES_DEV" device="" value="1K"/>
@@
 <instance part="Q3" gate="G$1" x="220.98" y="157.48" rot="R270"/>
 <instance part="R27" gate="G$1" x="213.36" y="160.02"/>
-<instance part="R29" gate="G$1" x="241.3" y="144.78" smashed="yes">
-<attribute name="NAME" x="235.712" y="145.542" size="1.27" layer="94"/>
-<attribute name="VALUE" x="242.57" y="145.288" size="1.27" layer="94"/>
-</instance>
-<instance part="R30" gate="G$1" x="236.22" y="142.24" smashed="yes">
-<attribute name="NAME" x="230.378" y="143.002" size="1.27" layer="94"/>
-<attribute name="VALUE" x="236.982" y="142.748" size="1.27" layer="94"/>
-</instance>
 <instance part="Q4" gate="G$1" x="190.5" y="119.38" smashed="yes" rot="R270">
 <attribute name="NAME" x="193.04" y="119.38" size="0.762" layer="94" rot="R270"/>
@@
 </segment>
 </net>
-<net name="N$39" class="0">
-<segment>
-<pinref part="J1" gate="G$1" pin="P$3"/>
-<pinref part="R30" gate="G$1" pin="P$2"/>
-<wire x1="246.38" y1="142.24" x2="238.76" y2="142.24" width="0.1524" layer="91"/>
-</segment>
-</net>
-<net name="N$40" class="0">
-<segment>
+<net name="DMX-" class="0">
+<segment>
+<wire x1="246.38" y1="144.78" x2="228.6" y2="144.78" width="0.1524" layer="91"/>
+<label x="228.6" y="144.78" size="1.6764" layer="95" rot="R180" xref="yes"/>
 <pinref part="J1" gate="G$1" pin="P$2"/>
-<pinref part="R29" gate="G$1" pin="P$2"/>
-<wire x1="246.38" y1="144.78" x2="243.84" y2="144.78" width="0.1524" layer="91"/>
-</segment>
-</net>
-<net name="DMX-" class="0">
-<segment>
-<pinref part="R29" gate="G$1" pin="P$1"/>
-<wire x1="238.76" y1="144.78" x2="228.6" y2="144.78" width="0.1524" layer="91"/>
-<label x="228.6" y="144.78" size="1.6764" layer="95" rot="R180" xref="yes"/>
 </segment>
 <segment>
@@
 <net name="DMX+" class="0">
 <segment>
-<pinref part="R30" gate="G$1" pin="P$1"/>
-<wire x1="233.68" y1="142.24" x2="220.98" y2="142.24" width="0.1524" layer="91"/>
+<wire x1="246.38" y1="142.24" x2="220.98" y2="142.24" width="0.1524" layer="91"/>
 <label x="220.98" y="142.24" size="1.6764" layer="95" rot="R180" xref="yes"/>
-</segment>
-<segment>
+<pinref part="J1" gate="G$1" pin="P$3"/>
+</segment>
+<segment>
